File: ShiftRegisterModule.brd (EAGLE design)
At the start: 22.9 x 15.2 mm, 6 parts, among them IC1 74595

Commit message: Mode board and schematic consistent
Parts:
- JP1: value (none) -> Outputs
- JP2: value (none) -> Inputs
- R1: value 1K5 -> 2K2
Changed lines of the file:
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@@
 <?xml version="1.0" encoding="utf-8"?>
 <!DOCTYPE eagle SYSTEM "eagle.dtd">
-<eagle version="6.5.0">
+<eagle version="9.3.0">
 <drawing>
 <settings>
-<setting alwaysvectorfont="yes"/>
+<setting alwaysvectorfont="no"/>
+<setting keepoldvectorfont="yes"/>
 <setting verticaltext="up"/>
 </settings>
@@
 <param name="dpMaxLengthDifference" value="10mm"/>
 <param name="dpGapFactor" value="2.5"/>
-<param name="checkGrid" value="0"/>
 <param name="checkAngle" value="0"/>
 <param name="checkFont" value="1"/>
 <param name="checkRestrict" value="1"/>
+<param name="checkStop" value="0"/>
+<param name="checkValues" value="0"/>
+<param name="checkNames" value="1"/>
+<param name="checkWireStubs" value="1"/>
+<param name="checkPolygonWidth" value="0"/>
 <param name="useDiameter" value="13"/>
 <param name="maxErrors" value="50"/>
@@
 <pass name="Default">
 <param name="RoutingGrid" value="50mil"/>
+<param name="AutoGrid" value="1"/>
+<param name="Efforts" value="0"/>
+<param name="TopRouterVariant" value="1"/>
 <param name="tpViaShape" value="round"/>
 <param name="PrefDir.1" value="|"/>
@@
 </autorouter>
 <elements>
-<element name="R1" library="freetronics-master-v1" package="0603" value="1K5" x="19.812" y="9.398" smashed="yes" rot="R180">
+<element name="R1" library="freetronics-master-v1" package="0603" value="2K2" x="19.812" y="9.398" smashed="yes" rot="R180">
 <attribute name="NAME" x="20.955" y="9.144" size="0.4064" layer="25" font="vector"/>
 <attribute name="VALUE" x="20.828" y="10.3632" size="0.4064" layer="27" font="vector" rot="R180"/>
@@
 <attribute name="VALUE" x="5.969" y="6.096" size="0.6096" layer="27" rot="R90"/>
 </element>
-<element name="JP1" library="freetronics-master-v1" package="1X08" value="" x="2.54" y="2.54" smashed="yes">
+<element name="JP1" library="freetronics-master-v1" package="1X08" value="Outputs" x="2.54" y="2.54" smashed="yes">
 <attribute name="NAME" x="2.7178" y="1.8288" size="1.27" layer="25" ratio="10"/>
 <attribute name="VALUE" x="1.27" y="-0.635" size="1.27" layer="27"/>
 </element>
-<element name="JP2" library="freetronics-master-v1" package="1X08" value="" x="2.54" y="12.7" smashed="yes">
+<element name="JP2" library="freetronics-master-v1" package="1X08" value="Inputs" x="2.54" y="12.7" smashed="yes">
 <attribute name="NAME" x="2.7178" y="12.2428" size="1.27" layer="25" ratio="10"/>
 <attribute name="VALUE" x="1.27" y="9.525" size="1.27" layer="27"/>
 </element>
-<element name="C1" library="freetronics-master-v1.1" package="0603" value="100nF" x="1.27" y="7.62" rot="R270"/>
+<element name="C1" library="freetronics-master-v1.1" package="0603" value="100nF" x="1.27" y="7.62" smashed="yes" rot="R270">
+<attribute name="NAME" x="1.778" y="8.509" size="0.4064" layer="25" font="vector" rot="R270"/>
+<attribute name="VALUE" x="0.3048" y="8.636" size="0.4064" layer="27" font="vector" rot="R270"/>
+</element>
 </elements>
 <signals>
@@
 </signal>
 </signals>
+<mfgpreviewcolors>
+<mfgpreviewcolor name="soldermaskcolor" color="0xC8008000"/>
+<mfgpreviewcolor name="silkscreencolor" color="0xFFFEFEFE"/>
+<mfgpreviewcolor name="backgroundcolor" color="0xFF282828"/>
+<mfgpreviewcolor name="coppercolor" color="0xFFFFBF00"/>
+<mfgpreviewcolor name="substratecolor" color="0xFF786E46"/>
+</mfgpreviewcolors>
 </board>
 </drawing>
